File: hardware/autoStart.kicad_sch (KiCad schematic)
At the start: 20 parts, among them J1 AudioJack3_Switch, J2 Screw_Terminal_01x03, Q1 BC547, U1 ICL7621BMTV, U2 LM7805

Commit message: Project prepared for converting to SMD
Parts:
- C2, C3: footprint (none) -> Capacitor_THT:C_Disc_D3.8mm_W2.6mm_P2.50mm
- J1: footprint connectors:ASJ195LHT -> Local_Connectors:AUDIO_JACK_ASJ-195-L-HT; symbol Connectors:AudioJack3_Switch -> Local_Connectors_Library:AudioJack3_Switch
- U1: symbol Operational_Amplifires:ICL7621BMTV -> Local_Miscellaneous_Library:ICL7621BMTV
- U2: renamed from U1; symbol Operational_Amplifires:ICL7621BMTV -> Local_Miscellaneous_Library:ICL7621BMTV
- U3: renamed from U2; value LM7805 -> 78S05M; footprint Package_TO_SOT_THT:TO-220-3_Vertical -> Package_TO_SOT_SMD:SOT-89-3; JLCPCB Part # (none) -> C400136; Manufacturer (none) -> UNI-SEMI
Changed lines of the file:
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@@
   (junction (at 93.98 109.22) (diameter 0) (color 0 0 0 0)
-  )
-  (junction (at 118.11 106.68) (diameter 0) (color 0 0 0 0)
   )
   (junction (at 198.12 76.2) (diameter 0) (color 0 0 0 0)
@@
     (stroke (width 0) (type default) (color 0 0 0 0))
   )
-  (wire (pts (xy 109.22 106.68) (xy 118.11 106.68))
-    (stroke (width 0) (type default) (color 0 0 0 0))
-  )
   (wire (pts (xy 163.83 82.55) (xy 163.83 111.76))
     (stroke (width 0) (type default) (color 0 0 0 0))
@@
       (effects (font (size 1.27 1.27)) (justify left))
     )
-    (property "Footprint" "" (id 2) (at 147.0152 121.92 0)
+    (property "Footprint" "Capacitor_THT:C_Disc_D3.8mm_W2.6mm_P2.50mm" (id 2) (at 147.0152 121.92 0)
       (effects (font (size 1.27 1.27)) hide)
     )
@@
     (property "Reference" "C2" (id 0) (at 130.81 100.5545 90))
     (property "Value" "100nf" (id 1) (at 130.81 103.3296 90))
-    (property "Footprint" "" (id 2) (at 134.62 105.7148 0)
+    (property "Footprint" "Capacitor_THT:C_Disc_D3.8mm_W2.6mm_P2.50mm" (id 2) (at 134.62 105.7148 0)
       (effects (font (size 1.27 1.27)) hide)
     )
@@
     (pin "2")
   )
-  (symbol (lib_id "Operational_Amplifires:ICL7621BMTV") (at 173.99 109.22 0) (unit 2)
+  (symbol (lib_id "Local_Miscellaneous_Library:ICL7621BMTV") (at 173.99 109.22 0) (unit 2)
     (in_bom yes) (on_board yes)
-    (property "Reference" "U1" (id 0) (at 177.8 100.33 0))
-    (property "Value" "ICL7621BMTV" (id 1) (at 177.8 102.87 0))
+    (property "Reference" "U1" (id 0) (at 173.99 104.14 0)
+      (effects (font (size 1.27 1.27)) (justify left))
+    )
+    (property "Value" "ICL7621BMTV" (id 1) (at 173.99 114.3 0)
+      (effects (font (size 1.27 1.27)) (justify left))
+    )
     (property "Footprint" "Package_TO_SOT_THT:TO-99-8" (id 2) (at 173.99 109.22 0)
       (effects (font (size 1.27 1.27)) hide)
@@
     (pin "1")
   )
-  (symbol (lib_id "Connectors:AudioJack3_Switch") (at 73.66 96.52 0) (unit 1)
-    (in_bom yes) (on_board yes) (fields_autoplaced)
-    (property "Reference" "J1" (id 0) (at 71.8185 87.4735 0))
-    (property "Value" "AudioJack3_Switch" (id 1) (at 71.8185 90.2486 0))
-    (property "Footprint" "connectors:ASJ195LHT" (id 2) (at 73.66 96.52 0)
+  (symbol (lib_id "Local_Connectors_Library:AudioJack3_Switch") (at 73.66 96.52 0) (unit 1)
+    (in_bom yes) (on_board yes) (fields_autoplaced)
+    (property "Reference" "J1" (id 0) (at 73.66 87.63 0))
+    (property "Value" "AudioJack3_Switch" (id 1) (at 73.66 90.17 0))
+    (property "Footprint" "Local_Connectors:AUDIO_JACK_ASJ-195-L-HT" (id 2) (at 73.66 96.52 0)
       (effects (font (size 1.27 1.27)) hide)
     )
@@
       (effects (font (size 1.27 1.27)) hide)
     )
+    (property "Description" "3,50mm (0,141\", 1/8\", ministik) - hovedtelefon Telefonhunstik Stereo (3 ledere, TRS) Stikforbindelse Loddemetal" (id 4) (at 73.66 96.52 0))
     (pin "1")
     (pin "2")
@@
     (pin "1")
   )
-  (symbol (lib_id "Operational_Amplifires:ICL7621BMTV") (at 110.49 106.68 0) (unit 1)
+  (symbol (lib_id "Local_Miscellaneous_Library:ICL7621BMTV") (at 110.49 106.68 0) (unit 1)
     (in_bom yes) (on_board yes)
-    (property "Reference" "U1" (id 0) (at 115.57 99.06 0))
-    (property "Value" "ICL7621BMTV" (id 1) (at 116.84 101.6 0))
+    (property "Reference" "U1" (id 0) (at 110.49 101.6 0)
+      (effects (font (size 1.27 1.27)) (justify left))
+    )
+    (property "Value" "ICL7621BMTV" (id 1) (at 110.49 111.76 0)
+      (effects (font (size 1.27 1.27)) (justify left))
+    )
     (property "Footprint" "Package_TO_SOT_THT:TO-99-8" (id 2) (at 110.49 106.68 0)
       (effects (font (size 1.27 1.27)) hide)
@@
     (pin "2")
   )
-  (symbol (lib_id "Operational_Amplifires:ICL7621BMTV") (at 110.49 106.68 0) (unit 3)
-    (in_bom yes) (on_board yes) (fields_autoplaced)
-    (property "Reference" "U1" (id 0) (at 108.585 107.159 0)
-      (effects (font (size 1.27 1.27)) (justify left) hide)
-    )
-    (property "Value" "ICL7621BMTV" (id 1) (at 108.585 108.5466 0)
-      (effects (font (size 1.27 1.27)) (justify left) hide)
+  (symbol (lib_id "Local_Miscellaneous_Library:ICL7621BMTV") (at 110.49 106.68 0) (unit 3)
+    (in_bom yes) (on_board yes) (fields_autoplaced)
+    (property "Reference" "U2" (id 0) (at 110.49 101.6 0)
+      (effects (font (size 1.27 1.27)) (justify left))
+    )
+    (property "Value" "ICL7621BMTV" (id 1) (at 110.49 111.76 0)
+      (effects (font (size 1.27 1.27)) (justify left))
     )
     (property "Footprint" "Package_TO_SOT_THT:TO-99-8" (id 2) (at 110.49 106.68 0)
@@
   (symbol (lib_id "Regulator_Linear:LM7805_TO220") (at 187.96 76.2 0) (mirror y) (unit 1)
     (in_bom yes) (on_board yes) (fields_autoplaced)
-    (property "Reference" "U2" (id 0) (at 187.96 70.3285 0))
-    (property "Value" "LM7805" (id 1) (at 187.96 73.1036 0))
-    (property "Footprint" "Package_TO_SOT_THT:TO-220-3_Vertical" (id 2) (at 187.96 70.485 0)
+    (property "Reference" "U3" (id 0) (at 187.96 70.3285 0))
+    (property "Value" "78S05M" (id 1) (at 187.96 73.1036 0))
+    (property "Footprint" "Package_TO_SOT_SMD:SOT-89-3" (id 2) (at 187.96 70.485 0)
       (effects (font (size 1.27 1.27) italic) hide)
     )
-    (property "Datasheet" "https://www.onsemi.cn/PowerSolutions/document/MC7800-D.PDF" (id 3) (at 187.96 77.47 0)
+    (property "Datasheet" "https://datasheet.lcsc.com/lcsc/1912111437_UNI-SEMI-78S05M_C400136.pdf" (id 3) (at 187.96 77.47 0)
+      (effects (font (size 1.27 1.27)) hide)
+    )
+    (property "Manufacturer" "UNI-SEMI" (id 4) (at 187.96 76.2 0)
+      (effects (font (size 1.27 1.27)) hide)
+    )
+    (property "JLCPCB Part #" "C400136" (id 5) (at 187.96 76.2 0)
       (effects (font (size 1.27 1.27)) hide)
     )
@@
     )
     (path "/7b485fa8-406a-42d5-9a01-13ae76ec07b5"
-      (reference "C2") (unit 1) (value "100nf") (footprint "")
+      (reference "C2") (unit 1) (value "100nf") (footprint "Capacitor_THT:C_Disc_D3.8mm_W2.6mm_P2.50mm")
     )
     (path "/28402017-1373-4e9f-83bc-1dd8451e4b54"
-      (reference "C3") (unit 1) (value "100nf") (footprint "")
+      (reference "C3") (unit 1) (value "100nf") (footprint "Capacitor_THT:C_Disc_D3.8mm_W2.6mm_P2.50mm")
     )
     (path "/eadbd981-3871-4a5e-b0f6-150a44ad3638"
@@
     )
     (path "/a87b0f82-053d-4565-9725-893652a134ac"
-      (reference "J1") (unit 1) (value "AudioJack3_Switch") (footprint "connectors:ASJ195LHT")
+      (reference "J1") (unit 1) (value "AudioJack3_Switch") (footprint "Local_Connectors:AUDIO_JACK_ASJ-195-L-HT")
     )
     (path "/b82d50c0-6690-4d03-8e11-7c35a4abeefa"
@@
     )
     (path "/ec0022a3-b763-4968-bab2-da03f869dff4"
-      (reference "U1") (unit 3) (value "ICL7621BMTV") (footprint "Package_TO_SOT_THT:TO-99-8")
+      (reference "U2") (unit 3) (value "ICL7621BMTV") (footprint "Package_TO_SOT_THT:TO-99-8")
     )
     (path "/eee40991-bfad-494f-89cf-cff149d4e6b0"
-      (reference "U2") (unit 1) (value "LM7805") (footprint "Package_TO_SOT_THT:TO-220-3_Vertical")
-    )
-  )
+      (reference "U3") (unit 1) (value "78S05M") (footprint "Package_TO_SOT_SMD:SOT-89-3")
+    )
+  )

Commit message: Final THT Mount commit
Parts:
- added J?: Conn_01x03_Male, symbol Connector:Conn_01x03_Male
Connections:
- net GND: now also J?.1 (Pin_1)
- net VS: now also J?.3 (Pin_3)
- net at J2.2 (Pin_2), Q1.1 (C): now also J?.2 (Pin_2)
Other:
- moved on the sheet: J2
Changed lines of the file:
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@@
     (company "El-Tek Trafikteknik I/S")
   )
+  (junction (at 208.28 100.33) (diameter 0) (color 0 0 0 0)
+  )
   (junction (at 146.05 106.68) (diameter 0) (color 0 0 0 0)
   )
@@
   (junction (at 146.05 125.73) (diameter 0) (color 0 0 0 0)
   )
+  (junction (at 208.28 102.87) (diameter 0) (color 0 0 0 0)
+  )
   (junction (at 154.94 125.73) (diameter 0) (color 0 0 0 0)
   )
@@
   )
   (junction (at 163.83 111.76) (diameter 0) (color 0 0 0 0)
+  )
+  (junction (at 208.28 97.79) (diameter 0) (color 0 0 0 0)
   )
   (junction (at 100.33 93.98) (diameter 0) (color 0 0 0 0)
@@
     (stroke (width 0) (type default) (color 0 0 0 0))
   )
-  (wire (pts (xy 198.12 104.14) (xy 208.28 104.14))
-    (stroke (width 0) (type default) (color 0 0 0 0))
-  )
   (wire (pts (xy 78.74 99.06) (xy 88.9 99.06))
     (stroke (width 0) (type default) (color 0 0 0 0))
   )
-  (wire (pts (xy 208.28 76.2) (xy 208.28 101.6))
+  (wire (pts (xy 208.28 76.2) (xy 208.28 97.79))
+    (stroke (width 0) (type default) (color 0 0 0 0))
+  )
+  (wire (pts (xy 208.28 100.33) (xy 198.12 100.33))
     (stroke (width 0) (type default) (color 0 0 0 0))
   )
@@
     (stroke (width 0) (type default) (color 0 0 0 0))
   )
+  (wire (pts (xy 198.12 100.33) (xy 198.12 104.14))
+    (stroke (width 0) (type default) (color 0 0 0 0))
+  )
   (wire (pts (xy 163.83 111.76) (xy 166.37 111.76))
     (stroke (width 0) (type default) (color 0 0 0 0))
@@
     (stroke (width 0) (type default) (color 0 0 0 0))
   )
-  (wire (pts (xy 208.28 125.73) (xy 208.28 106.68))
+  (wire (pts (xy 208.28 125.73) (xy 208.28 102.87))
     (stroke (width 0) (type default) (color 0 0 0 0))
   )
@@
     (stroke (width 0) (type default) (color 0 0 0 0))
   )
+  (wire (pts (xy 208.28 102.87) (xy 224.79 102.87))
+    (stroke (width 0) (type default) (color 0 0 0 0))
+  )
+  (wire (pts (xy 208.28 97.79) (xy 224.79 97.79))
+    (stroke (width 0) (type default) (color 0 0 0 0))
+  )
   (wire (pts (xy 146.05 106.68) (xy 146.05 114.3))
     (stroke (width 0) (type default) (color 0 0 0 0))
@@
   )
   (wire (pts (xy 78.74 104.14) (xy 80.01 104.14))
+    (stroke (width 0) (type default) (color 0 0 0 0))
+  )
+  (wire (pts (xy 208.28 100.33) (xy 224.79 100.33))
     (stroke (width 0) (type default) (color 0 0 0 0))
   )
@@
     (pin "2")
   )
+  (symbol (lib_id "Connector:Conn_01x03_Male") (at 229.87 100.33 180) (unit 1)
+    (in_bom yes) (on_board yes) (fields_autoplaced)
+    (property "Reference" "J?" (id 0) (at 230.5812 99.4215 0)
+      (effects (font (size 1.27 1.27)) (justify right))
+    )
+    (property "Value" "Conn_01x03_Male" (id 1) (at 230.5812 102.1966 0)
+      (effects (font (size 1.27 1.27)) (justify right))
+    )
+    (property "Footprint" "" (id 2) (at 229.87 100.33 0)
+      (effects (font (size 1.27 1.27)) hide)
+    )
+    (property "Datasheet" "~" (id 3) (at 229.87 100.33 0)
+      (effects (font (size 1.27 1.27)) hide)
+    )
+    (pin "1")
+    (pin "2")
+    (pin "3")
+  )
   (symbol (lib_id "power:VS") (at 219.71 74.93 0) (mirror x) (unit 1)
     (in_bom yes) (on_board yes) (fields_autoplaced)
@@
     (pin "2")
   )
-  (symbol (lib_id "Connector:Screw_Terminal_01x03") (at 213.36 104.14 0) (mirror x) (unit 1)
-    (in_bom yes) (on_board yes) (fields_autoplaced)
-    (property "Reference" "J2" (id 0) (at 213.36 96.3635 0))
-    (property "Value" "Screw_Terminal_01x03" (id 1) (at 213.36 99.1386 0))
-    (property "Footprint" "TerminalBlock_Phoenix:TerminalBlock_Phoenix_MKDS-1,5-3_1x03_P5.00mm_Horizontal" (id 2) (at 213.36 104.14 0)
-      (effects (font (size 1.27 1.27)) hide)
-    )
-    (property "Datasheet" "~" (id 3) (at 213.36 104.14 0)
+  (symbol (lib_id "Connector:Screw_Terminal_01x03") (at 213.36 100.33 0) (mirror x) (unit 1)
+    (in_bom yes) (on_board yes) (fields_autoplaced)
+    (property "Reference" "J2" (id 0) (at 213.36 92.5535 0))
+    (property "Value" "Screw_Terminal_01x03" (id 1) (at 213.36 95.3286 0))
+    (property "Footprint" "TerminalBlock_Phoenix:TerminalBlock_Phoenix_MKDS-1,5-3_1x03_P5.00mm_Horizontal" (id 2) (at 213.36 100.33 0)
+      (effects (font (size 1.27 1.27)) hide)
+    )
+    (property "Datasheet" "~" (id 3) (at 213.36 100.33 0)
       (effects (font (size 1.27 1.27)) hide)
     )
@@
       (reference "J2") (unit 1) (value "Screw_Terminal_01x03") (footprint "TerminalBlock_Phoenix:TerminalBlock_Phoenix_MKDS-1,5-3_1x03_P5.00mm_Horizontal")
     )
+    (path "/9a3519d7-ebfa-46a5-a572-5252a6310af5"
+      (reference "J?") (unit 1) (value "Conn_01x03_Male") (footprint "")
+    )
     (path "/0b739a5d-c787-4f6f-8edd-9626528c59c7"

Commit message: SMD Mounts Initial commit
Parts:
- removed C1: 10nf, Capacitor_THT:C_Disc_D4.3mm_W1.9mm_P5.00mm, symbol Device:C
- removed C2, C3: 100nf, Capacitor_THT:C_Disc_D3.8mm_W2.6mm_P2.50mm, symbol Device:C
- removed C4: 0,1uf, Capacitor_THT:CP_Radial_Tantal_D5.0mm_P5.00mm, symbol Device:C_Polarized_Small
- removed C5: 0,47uf, Capacitor_THT:CP_Radial_Tantal_D5.0mm_P5.00mm, symbol Device:C_Polarized_Small
- removed D1: 1N4148, Diode_THT:D_DO-35_SOD27_P7.62mm_Horizontal, symbol Diode:1N4148
- removed J2: Screw_Terminal_01x03, TerminalBlock_Phoenix:TerminalBlock_Phoenix_MKDS-1,5-3_1x03_P5.00mm_Horizontal, symbol Connector:Screw_Terminal_01x03
- removed J?: Conn_01x03_Male, symbol Connector:Conn_01x03_Male
- removed Q1: BC547, Package_TO_SOT_THT:TO-92L_Inline_Wide, symbol Transistor_BJT:BC547
- removed R1, R2, R3: 10k, Resistor_THT:R_Axial_DIN0411_L9.9mm_D3.6mm_P12.70mm_Horizontal, symbol Device:R
- removed R4: 330k, Resistor_THT:R_Axial_DIN0411_L9.9mm_D3.6mm_P12.70mm_Horizontal, symbol Device:R
- removed R5: 100k, Resistor_THT:R_Axial_DIN0411_L9.9mm_D3.6mm_P12.70mm_Horizontal, symbol Device:R
- removed R6: 680k, Resistor_THT:R_Axial_DIN0411_L9.9mm_D3.6mm_P12.70mm_Horizontal, symbol Device:R
- removed R7: 150k, Resistor_THT:R_Axial_DIN0411_L9.9mm_D3.6mm_P12.70mm_Horizontal, symbol Device:R
- removed R8: 33k, Resistor_THT:R_Axial_DIN0411_L9.9mm_D3.6mm_P12.70mm_Horizontal, symbol Device:R
- removed R9: 180, Resistor_THT:R_Axial_DIN0411_L9.9mm_D3.6mm_P12.70mm_Horizontal, symbol Device:R
- removed U1, U2: ICL7621BMTV, Package_TO_SOT_THT:TO-99-8, symbol Local_Miscellaneous_Library:ICL7621BMTV
- removed U3: 78S05M, Package_TO_SOT_SMD:SOT-89-3, symbol Regulator_Linear:LM7805_TO220
- added C1: C10nf_SMD, Capacitor_SMD:C_0402_1005Metric, symbol Local_Device_Library:C10nf_SMD
- added C2, C3, C4: C100nf_SMD, Capacitor_SMD:C_0402_1005Metric, symbol Local_Device_Library:C100nf_SMD
- added C5: C330nf_SMD, Capacitor_SMD:C_0805_2012Metric, symbol Local_Device_Library:C330nf_SMD
- added D1: 1N4148WS, Diode_SMD:D_SOD-323F, symbol Local_Diode_Library:1N4148WS
- added J2: Screw_Terminal_01x03-Connector, Local_Connectors:Phoenix_TERM_BLOCK_3POS_45DEG_5MM_PCB, symbol Local_Connectors_Library:Screw_Terminal_01x03-Connector
- added J3: Conn_01x03_Male, Local_Project_Connectors_Library:PinHeader_1x03_P_5mm_Vertical-(Backside_Mount), symbol Connector:Conn_01x03_Male
- added Q1: S8050_SOT23, Package_TO_SOT_SMD:SOT-23, symbol Local_Transistor_BJT_Library:S8050_SOT23
- added R1, R2, R3: R10K_0.0625W, Resistor_SMD:R_0402_1005Metric, symbol Local_Device_Library:R10K_0.0625W
- added R4: R330K_0.0625W, Resistor_SMD:R_0402_1005Metric, symbol Local_Device_Library:R330K_0.0625W
- added R5: R100K_0.0625W, Resistor_SMD:R_0402_1005Metric, symbol Local_Device_Library:R100K_0.0625W
- added R6: R680K_0.1W, Resistor_SMD:R_0201_0603Metric, symbol Local_Device_Library:R680K_0.1W
- added R7: R150K_0.0625W, Resistor_SMD:R_0402_1005Metric, symbol Local_Device_Library:R150K_0.0625W
- added R8: R33K_0.0625W, Resistor_SMD:R_0402_1005Metric, symbol Local_Device_Library:R33K_0.0625W
- added R9: R180_0.125W, Resistor_SMD:R_0805_2012Metric, symbol Local_Device_Library:R180_0.125W
- added U1: LM358DR2G, Package_SO:SOIC-8_3.9x4.9mm_P1.27mm, symbol Local_Miscellaneous_Library:LM358DR2G
- added U2: 78L05G_SOT89, Package_TO_SOT_SMD:SOT-89-3, symbol Local_Miscellaneous_Library:78L05G_SOT89
- J1: footprint Local_Connectors:AUDIO_JACK_ASJ-195-L-HT -> Local_Connectors:AUDIO_JACK_ASJ-195-L-HT-(Backside_Mount)
Connections:
- net GND: now also C3.2, C4.2, C5.2, J2.1 (Pin_1), J3.1 (Pin_1), Q1.2 (E), R3.2, R5.2, R6.2, R8.2, U1.4 (V-), U2.2 (GND)
- net VCC: now also C4.1, R2.1, R7.1, U1.8 (V+), U2.1 (OUT)
- net VS: now also C5.1, J2.3 (Pin_3), J3.3 (Pin_3), U2.3 (IN)
- net at J1.2 (T): now also R2.2, R3.1, U1.6 (-)
- net at J1.1 (S): now also R1.1
- new net: C1.1, R1.2, R4.1, U1.5 (+)
- new net: C1.2, C2.1, R4.2, U1.7
- new net: C2.2, D1.2 (A), R5.1
- new net: R7.2, R8.1, U1.2 (-)
- new net: J2.2 (Pin_2), J3.2 (Pin_2), Q1.3 (C)
- new net: C3.1, D1.1 (K), R6.1, U1.3 (+)
- new net: Q1.1 (B), R9.2
- new net: R9.1, U1.1
